Commit message: adding the new model, doesn't work for now

File: urdf/demo.urdf.xacro (robot description, xacro)
@@ -4,5 +4,5 @@
   <xacro:include filename="$(find panda_torque_mpc)/urdf/support.urdf.xacro"/>
   <xacro:support/>
-  <xacro:franka_robot arm_id="panda2"
+  <xacro:franka_robot arm_id="panda"
                       joint_limits="${xacro.load_yaml('$(find franka_description)/robots/panda/joint_limits.yaml')}">
   </xacro:franka_robot>

File: urdf/robot-gazebo.urdf (robot description, URDF)
Before this commit: robot pandas, 41 links, 40 joints
Links:
- removed link panda2_camera_support_link
- removed link panda2_hand
- removed link panda2_hand_sc
- removed link panda2_hand_tcp
- removed link panda2_leftfinger
- removed link panda2_link0
- removed link panda2_link0_sc
- removed link panda2_link1
- removed link panda2_link1_sc
- removed link panda2_link2
- removed link panda2_link2_sc
- removed link panda2_link3
- removed link panda2_link3_sc
- removed link panda2_link4
- removed link panda2_link4_sc
- removed link panda2_link5
- removed link panda2_link5_sc
- removed link panda2_link6
- removed link panda2_link6_sc
- removed link panda2_link7
- removed link panda2_link7_sc
- removed link panda2_link8
- removed link panda2_ref_camera_link
- removed link panda2_rightfinger
- added link panda_camera_support_link, mass 0.010; collision mesh filename=package://panda_torque_mpc/meshes/camera-support.stl scale=1 1 1; visual mesh filename=package://panda_torque_mpc/meshes/camera-support.stl scale=1 1 1
- added link panda_hand, mass 0.73; collision mesh filename=package://franka_description/meshes/collision/hand.stl; visual mesh filename=package://franka_description/meshes/visual/hand.dae
- added link panda_hand_sc
- added link panda_hand_tcp
- added link panda_leftfinger, mass 0.015; collision box size=17.5e-3 15.2e-3 18.5e-3; collision box size=17.5e-3 7e-3 23.5e-3
- added link panda_link0, mass 0.629769; collision mesh filename=package://franka_description/meshes/collision/link0.stl; visual mesh filename=package://franka_description/meshes/visual/link0.dae
- added link panda_link0_sc
- added link panda_link1, mass 4.970684; collision mesh filename=package://franka_description/meshes/collision/link1.stl; visual mesh filename=package://franka_description/meshes/visual/link1.dae
- added link panda_link1_sc
- added link panda_link2, mass 0.646926; collision mesh filename=package://franka_description/meshes/collision/link2.stl; visual mesh filename=package://franka_description/meshes/visual/link2.dae
- added link panda_link2_sc
- added link panda_link3, mass 3.228604; collision mesh filename=package://franka_description/meshes/collision/link3.stl; visual mesh filename=package://franka_description/meshes/visual/link3.dae
- added link panda_link3_sc
- added link panda_link4, mass 3.587895; collision mesh filename=package://franka_description/meshes/collision/link4.stl; visual mesh filename=package://franka_description/meshes/visual/link4.dae
- added link panda_link4_sc
- added link panda_link5, mass 1.225946; collision mesh filename=package://franka_description/meshes/collision/link5.stl; visual mesh filename=package://franka_description/meshes/visual/link5.dae
- added link panda_link5_sc
- added link panda_link6, mass 1.666555; collision mesh filename=package://franka_description/meshes/collision/link6.stl; visual mesh filename=package://franka_description/meshes/visual/link6.dae
- added link panda_link6_sc
- added link panda_link7, mass 0.735522; collision mesh filename=package://franka_description/meshes/collision/link7.stl; visual mesh filename=package://franka_description/meshes/visual/link7.dae
- added link panda_link7_sc
- added link panda_link8
- added link panda_ref_camera_link
- added link panda_rightfinger, mass 0.015; collision box size=17.5e-3 15.2e-3 18.5e-3; collision box size=17.5e-3 7e-3 23.5e-3
Joints:
- removed joint panda2_camera_support_joint
- removed joint panda2_finger_joint1
- removed joint panda2_finger_joint2
- removed joint panda2_hand_joint
- removed joint panda2_hand_sc_joint
- removed joint panda2_hand_tcp_joint
- removed joint panda2_joint1
- removed joint panda2_joint2
- removed joint panda2_joint3
- removed joint panda2_joint4
- removed joint panda2_joint5
- removed joint panda2_joint6
- removed joint panda2_joint7
- removed joint panda2_joint8
- removed joint panda2_link0_sc_joint
- removed joint panda2_link1_sc_joint
- removed joint panda2_link2_sc_joint
- removed joint panda2_link3_sc_joint
- removed joint panda2_link4_sc_joint
- removed joint panda2_link5_sc_joint
- removed joint panda2_link6_sc_joint
- removed joint panda2_link7_sc_joint
- removed joint panda2_ref_camera_joint
- added joint panda_camera_support_joint: type fixed, parent panda_hand, child panda_camera_support_link, origin xyz=0 0 0 rpy=3.141592653589793 0 0
- added joint panda_finger_joint1: type prismatic, parent panda_hand, child panda_leftfinger, origin xyz=0 0 0.0584 rpy=0 0 0, axis 0 1 0, limit lower=0.0 upper=0.04 effort=100 velocity=0.2
- added joint panda_finger_joint2: type prismatic, parent panda_hand, child panda_rightfinger, origin xyz=0 0 0.0584 rpy=0 0 0, axis 0 -1 0, limit lower=0.0 upper=0.04 effort=100 velocity=0.2, mimic joint=panda_finger_joint1
- added joint panda_hand_joint: type fixed, parent panda_link8, child panda_hand, origin xyz=0 0 0 rpy=0 0 -0.7853981633974483
- added joint panda_hand_sc_joint: type fixed, parent panda_hand, child panda_hand_sc, origin rpy=0 0 0
- added joint panda_hand_tcp_joint: type fixed, parent panda_hand, child panda_hand_tcp, origin xyz=0 0 0.1034 rpy=0 0 0
- added joint panda_joint1: type revolute, parent panda_link0, child panda_link1, origin xyz=0 0 0.333 rpy=0 0 0, axis 0 0 1, limit lower=-2.8973 upper=2.8973 effort=87.0 velocity=2.175
- added joint panda_joint2: type revolute, parent panda_link1, child panda_link2, origin xyz=0 0 0 rpy=-1.5707963267948966 0 0, axis 0 0 1, limit lower=-1.7628 upper=1.7628 effort=87.0 velocity=2.175
- added joint panda_joint3: type revolute, parent panda_link2, child panda_link3, origin xyz=0 -0.316 0 rpy=1.5707963267948966 0 0, axis 0 0 1, limit lower=-2.8973 upper=2.8973 effort=87.0 velocity=2.175
- added joint panda_joint4: type revolute, parent panda_link3, child panda_link4, origin xyz=0.0825 0 0 rpy=1.5707963267948966 0 0, axis 0 0 1, limit lower=-3.0718 upper=-0.0698 effort=87.0 velocity=2.175
- added joint panda_joint5: type revolute, parent panda_link4, child panda_link5, origin xyz=-0.0825 0.384 0 rpy=-1.5707963267948966 0 0, axis 0 0 1, limit lower=-2.8973 upper=2.8973 effort=12.0 velocity=2.61
- added joint panda_joint6: type revolute, parent panda_link5, child panda_link6, origin xyz=0 0 0 rpy=1.5707963267948966 0 0, axis 0 0 1, limit lower=-0.0175 upper=3.7525 effort=12.0 velocity=2.61
- added joint panda_joint7: type revolute, parent panda_link6, child panda_link7, origin xyz=0.088 0 0 rpy=1.5707963267948966 0 0, axis 0 0 1, limit lower=-2.8973 upper=2.8973 effort=12.0 velocity=2.61
- added joint panda_joint8: type fixed, parent panda_link7, child panda_link8, origin xyz=0 0 0.107 rpy=0 0 0
- added joint panda_link0_sc_joint: type fixed, parent panda_link0, child panda_link0_sc, origin rpy=0 0 0
- added joint panda_link1_sc_joint: type fixed, parent panda_link1, child panda_link1_sc, origin rpy=0 0 0
- added joint panda_link2_sc_joint: type fixed, parent panda_link2, child panda_link2_sc, origin rpy=0 0 0
- added joint panda_link3_sc_joint: type fixed, parent panda_link3, child panda_link3_sc, origin rpy=0 0 0
- added joint panda_link4_sc_joint: type fixed, parent panda_link4, child panda_link4_sc, origin rpy=0 0 0
- added joint panda_link5_sc_joint: type fixed, parent panda_link5, child panda_link5_sc, origin rpy=0 0 0
- added joint panda_link6_sc_joint: type fixed, parent panda_link6, child panda_link6_sc, origin rpy=0 0 0
- added joint panda_link7_sc_joint: type fixed, parent panda_link7, child panda_link7_sc, origin rpy=0 0 0.7853981633974483
- added joint panda_ref_camera_joint: type fixed, parent panda_hand, child panda_ref_camera_link, origin xyz=0.13682768843416482                    -0.009443400298528096                    -0.08387833599341328 rpy=0.022100209841200636                    -1.3156624527412932                    3.061881150974905
- joint camera_joint: parent panda2_ref_camera_link -> panda_ref_camera_link
- joint support_joint: child panda2_link0 -> panda_link0

File: urdf/robot.urdf (robot description, URDF)
Before this commit: robot pandas, 41 links, 40 joints
Links:
- removed link panda2_camera_support_link
- removed link panda2_hand
- removed link panda2_hand_sc
- removed link panda2_hand_tcp
- removed link panda2_leftfinger
- removed link panda2_link0
- removed link panda2_link0_sc
- removed link panda2_link1
- removed link panda2_link1_sc
- removed link panda2_link2
- removed link panda2_link2_sc
- removed link panda2_link3
- removed link panda2_link3_sc
- removed link panda2_link4
- removed link panda2_link4_sc
- removed link panda2_link5
- removed link panda2_link5_sc
- removed link panda2_link6
- removed link panda2_link6_sc
- removed link panda2_link7
- removed link panda2_link7_sc
- removed link panda2_link8
- removed link panda2_ref_camera_link
- removed link panda2_rightfinger
- added link panda_camera_support_link, mass 0.010; collision mesh filename=package://panda_torque_mpc/meshes/camera-support.stl scale=1 1 1; visual mesh filename=package://panda_torque_mpc/meshes/camera-support.stl scale=1 1 1
- added link panda_hand; collision mesh filename=package://franka_description/meshes/collision/hand.stl; visual mesh filename=package://franka_description/meshes/visual/hand.dae
- added link panda_hand_sc
- added link panda_hand_tcp
- added link panda_leftfinger; collision box size=17.5e-3 15.2e-3 18.5e-3; collision box size=17.5e-3 7e-3 23.5e-3
- added link panda_link0; collision mesh filename=package://franka_description/meshes/collision/link0.stl; visual mesh filename=package://franka_description/meshes/visual/link0.dae
- added link panda_link0_sc; collision cylinder length=0.03 radius=0.09; collision sphere radius=0.09
- added link panda_link1; collision mesh filename=package://franka_description/meshes/collision/link1.stl; visual mesh filename=package://franka_description/meshes/visual/link1.dae
- added link panda_link1_sc; collision cylinder length=0.283 radius=0.09; collision sphere radius=0.09
- added link panda_link2; collision mesh filename=package://franka_description/meshes/collision/link2.stl; visual mesh filename=package://franka_description/meshes/visual/link2.dae
- added link panda_link2_sc; collision cylinder length=0.12 radius=0.09; collision sphere radius=0.09
- added link panda_link3; collision mesh filename=package://franka_description/meshes/collision/link3.stl; visual mesh filename=package://franka_description/meshes/visual/link3.dae
- added link panda_link3_sc; collision cylinder length=0.15 radius=0.09; collision sphere radius=0.09
- added link panda_link4; collision mesh filename=package://franka_description/meshes/collision/link4.stl; visual mesh filename=package://franka_description/meshes/visual/link4.dae
- added link panda_link4_sc; collision cylinder length=0.12 radius=0.09; collision sphere radius=0.09
- added link panda_link5; collision mesh filename=package://franka_description/meshes/collision/link5.stl; visual mesh filename=package://franka_description/meshes/visual/link5.dae
- added link panda_link5_sc; collision cylinder length=0.1 radius=0.09; collision cylinder length=0.14 radius=0.055
- added link panda_link6; collision mesh filename=package://franka_description/meshes/collision/link6.stl; visual mesh filename=package://franka_description/meshes/visual/link6.dae
- added link panda_link6_sc; collision cylinder length=0.08 radius=0.08; collision sphere radius=0.08
- added link panda_link7; collision mesh filename=package://franka_description/meshes/collision/link7.stl; visual mesh filename=package://franka_description/meshes/visual/link7.dae
- added link panda_link7_sc; collision cylinder length=0.01 radius=0.06; collision cylinder length=0.14 radius=0.07
- added link panda_link8
- added link panda_ref_camera_link
- added link panda_rightfinger; collision box size=17.5e-3 15.2e-3 18.5e-3; collision box size=17.5e-3 7e-3 23.5e-3
Joints:
- removed joint panda2_camera_support_joint
- removed joint panda2_finger_joint1
- removed joint panda2_finger_joint2
- removed joint panda2_hand_joint
- removed joint panda2_hand_sc_joint
- removed joint panda2_hand_tcp_joint
- removed joint panda2_joint1
- removed joint panda2_joint2
- removed joint panda2_joint3
- removed joint panda2_joint4
- removed joint panda2_joint5
- removed joint panda2_joint6
- removed joint panda2_joint7
- removed joint panda2_joint8
- removed joint panda2_link0_sc_joint
- removed joint panda2_link1_sc_joint
- removed joint panda2_link2_sc_joint
- removed joint panda2_link3_sc_joint
- removed joint panda2_link4_sc_joint
- removed joint panda2_link5_sc_joint
- removed joint panda2_link6_sc_joint
- removed joint panda2_link7_sc_joint
- removed joint panda2_ref_camera_joint
- added joint panda_camera_support_joint: type fixed, parent panda_hand, child panda_camera_support_link, origin xyz=0 0 0 rpy=3.141592653589793 0 0
- added joint panda_finger_joint1: type prismatic, parent panda_hand, child panda_leftfinger, origin xyz=0 0 0.0584 rpy=0 0 0, axis 0 1 0, limit lower=0.0 upper=0.04 effort=100 velocity=0.2
- added joint panda_finger_joint2: type prismatic, parent panda_hand, child panda_rightfinger, origin xyz=0 0 0.0584 rpy=0 0 0, axis 0 -1 0, limit lower=0.0 upper=0.04 effort=100 velocity=0.2, mimic joint=panda_finger_joint1
- added joint panda_hand_joint: type fixed, parent panda_link8, child panda_hand, origin xyz=0 0 0 rpy=0 0 -0.7853981633974483
- added joint panda_hand_sc_joint: type fixed, parent panda_hand, child panda_hand_sc, origin rpy=0 0 0
- added joint panda_hand_tcp_joint: type fixed, parent panda_hand, child panda_hand_tcp, origin xyz=0 0 0.1034 rpy=0 0 0
- added joint panda_joint1: type revolute, parent panda_link0, child panda_link1, origin xyz=0 0 0.333 rpy=0 0 0, axis 0 0 1, limit lower=-2.8973 upper=2.8973 effort=87.0 velocity=2.175
- added joint panda_joint2: type revolute, parent panda_link1, child panda_link2, origin xyz=0 0 0 rpy=-1.5707963267948966 0 0, axis 0 0 1, limit lower=-1.7628 upper=1.7628 effort=87.0 velocity=2.175
- added joint panda_joint3: type revolute, parent panda_link2, child panda_link3, origin xyz=0 -0.316 0 rpy=1.5707963267948966 0 0, axis 0 0 1, limit lower=-2.8973 upper=2.8973 effort=87.0 velocity=2.175
- added joint panda_joint4: type revolute, parent panda_link3, child panda_link4, origin xyz=0.0825 0 0 rpy=1.5707963267948966 0 0, axis 0 0 1, limit lower=-3.0718 upper=-0.0698 effort=87.0 velocity=2.175
- added joint panda_joint5: type revolute, parent panda_link4, child panda_link5, origin xyz=-0.0825 0.384 0 rpy=-1.5707963267948966 0 0, axis 0 0 1, limit lower=-2.8973 upper=2.8973 effort=12.0 velocity=2.61
- added joint panda_joint6: type revolute, parent panda_link5, child panda_link6, origin xyz=0 0 0 rpy=1.5707963267948966 0 0, axis 0 0 1, limit lower=-0.0175 upper=3.7525 effort=12.0 velocity=2.61
- added joint panda_joint7: type revolute, parent panda_link6, child panda_link7, origin xyz=0.088 0 0 rpy=1.5707963267948966 0 0, axis 0 0 1, limit lower=-2.8973 upper=2.8973 effort=12.0 velocity=2.61
- added joint panda_joint8: type fixed, parent panda_link7, child panda_link8, origin xyz=0 0 0.107 rpy=0 0 0
- added joint panda_link0_sc_joint: type fixed, parent panda_link0, child panda_link0_sc, origin rpy=0 0 0
- added joint panda_link1_sc_joint: type fixed, parent panda_link1, child panda_link1_sc, origin rpy=0 0 0
- added joint panda_link2_sc_joint: type fixed, parent panda_link2, child panda_link2_sc, origin rpy=0 0 0
- added joint panda_link3_sc_joint: type fixed, parent panda_link3, child panda_link3_sc, origin rpy=0 0 0
- added joint panda_link4_sc_joint: type fixed, parent panda_link4, child panda_link4_sc, origin rpy=0 0 0
- added joint panda_link5_sc_joint: type fixed, parent panda_link5, child panda_link5_sc, origin rpy=0 0 0
- added joint panda_link6_sc_joint: type fixed, parent panda_link6, child panda_link6_sc, origin rpy=0 0 0
- added joint panda_link7_sc_joint: type fixed, parent panda_link7, child panda_link7_sc, origin rpy=0 0 0.7853981633974483
- added joint panda_ref_camera_joint: type fixed, parent panda_hand, child panda_ref_camera_link, origin xyz=0.13682768843416482                    -0.009443400298528096                    -0.08387833599341328 rpy=0.022100209841200636                    -1.3156624527412932                    3.061881150974905
- joint camera_joint: parent panda2_ref_camera_link -> panda_ref_camera_link
- joint support_joint: child panda2_link0 -> panda_link0

File: urdf/support.urdf.xacro (robot description, xacro)
@@ -157,5 +157,5 @@
         <origin xyz="0.563 -0.1655 .78" rpy="0 0 ${pi}" />
         <parent link="support_link" />
-        <child  link="panda2_link0" />
+        <child  link="panda_link0" />
       </joint>
       <joint name="wall_joint_1" type="fixed">

Commit message: changes on URDF : Adding inertial parameters & adding Example Robot Data URDF in the urdf dir & changing names pandas to panda

File: urdf/demo.urdf.xacro (robot description, xacro)
@@ -1,4 +1,4 @@
 <?xml version='1.0' encoding='utf-8'?>
-<robot xmlns:xacro="http://www.ros.org/wiki/xacro" name="pandas">
+<robot xmlns:xacro="http://www.ros.org/wiki/xacro" name="panda">
   <xacro:include filename="$(find panda_torque_mpc)/urdf/franka_robot.xacro"/>
   <xacro:include filename="$(find panda_torque_mpc)/urdf/support.urdf.xacro"/>

File: urdf/robot.urdf (robot description, URDF)
Before this commit: robot pandas, 41 links, 40 joints
Links:
- link panda_hand: mass None -> 0.73; geometry collision mesh filename=package://example-robot-data/robots/panda_description/meshe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; visual mesh filename=package://example-robot-data/robots/panda_description/meshe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
- link panda_hand_tcp: mass None -> 0
- link panda_leftfinger: mass None -> 0.015; geometry collision box size=17.5e-3 15.2e-3 18.5e-3; collision box size=17.5e-3 7e-3 23.5e-3
- link panda_link0: mass None -> 0.629769; geometry collision mesh filename=package://example-robot-data/robots/panda_description/meshe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; visual mesh filename=package://example-robot-data/robots/panda_description/meshe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
- link panda_link1: mass None -> 4.970684; geometry collision mesh filename=package://example-robot-data/robots/panda_description/meshe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; visual mesh filename=package://example-robot-data/robots/panda_description/meshe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
- link panda_link2: mass None -> 0.646926; geometry collision mesh filename=package://example-robot-data/robots/panda_description/meshe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; visual mesh filename=package://example-robot-data/robots/panda_description/meshe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
- link panda_link3: mass None -> 3.228604; geometry collision mesh filename=package://example-robot-data/robots/panda_description/meshe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; visual mesh filename=package://example-robot-data/robots/panda_description/meshe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
- link panda_link4: mass None -> 3.587895; geometry collision mesh filename=package://example-robot-data/robots/panda_description/meshe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; visual mesh filename=package://example-robot-data/robots/panda_description/meshe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
- link panda_link5: mass None -> 1.225946; geometry collision mesh filename=package://example-robot-data/robots/panda_description/meshe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; visual mesh filename=package://example-robot-data/robots/panda_description/meshe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
- link panda_link6: mass None -> 1.666555; geometry collision mesh filename=package://example-robot-data/robots/panda_description/meshe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; visual mesh filename=package://example-robot-data/robots/panda_description/meshe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
- link panda_link7: mass None -> 0.735522; geometry collision mesh filename=package://example-robot-data/robots/panda_description/meshe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; visual mesh filename=package://example-robot-data/robots/panda_description/meshe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
- link panda_link8: mass None -> 0
- link panda_rightfinger: mass None -> 0.015; geometry collision box size=17.5e-3 15.2e-3 18.5e-3; collision box size=17.5e-3 7e-3 23.5e-3
