Commit message: adding a ros node for the warm start

File: urdf/robot.urdf (robot description, URDF)
Before this commit: robot panda, 41 links, 40 joints
Links:
- link panda_leftfinger: geometry collision sphere radius=.03; visual mesh filename=package://example-robot-data/robots/panda_description/meshe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
- link panda_rightfinger: geometry collision sphere radius=.03; visual mesh filename=package://example-robot-data/robots/panda_description/meshe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

File: urdf/support.urdf.xacro (robot description, xacro)
@@ -14,10 +14,10 @@
           </geometry>
         </visual>
-        <collision>
+        <!-- <collision>
           <origin xyz="0 0 0.38"/>
           <geometry>
 	    <box size="1.703 0.803 0.76"/>
           </geometry>
-        </collision>
+        </collision> -->
         <!--visual>
           <origin xyz="-0.61 0.2215 0.77"/>
@@ -38,8 +38,30 @@
           </geometry>
         </visual>
-        <collision>
+        <!-- <collision>
           <origin xyz="0.6385 -0.1655 0.77"/>
           <geometry>
             <box size="0.3 0.3 0.02"/>
+          </geometry>
+        </collision> -->
+      </link>
+      <link name="the_ball">
+        <inertial>
+          <mass value="1"/>
+          <origin xyz="0 0 0"/>
+          <inertia ixx="1"  ixy="0"  ixz="0" iyy="1" iyz="0" izz="1" />
+        </inertial>
+        <visual>
+          <origin xyz="0 0 0"/>
+          <geometry>
+            <sphere radius="0.15"/>
+          </geometry>
+          <material name="green">
+            <color rgba ="0 1 0 0.8"/>
+          </material>
+        </visual>
+        <collision>
+          <origin xyz="0 0 0"/>
+          <geometry>
+            <sphere radius="0.15"/>
           </geometry>
         </collision>
@@ -184,4 +206,9 @@
         <child link="panda1_box"/>
       </joint>
+      <joint name="the_ball_joint" type="fixed">
+        <origin xyz="0 0 0.8" />
+        <parent link="world"/>
+        <child link="the_ball"/>
+      </joint>
   </xacro:macro>
 </robot>
