Commit message: adding the meshes + updating the CMakeList + adding new URDF for pinocchio

File: urdf/franka_robot.xacro (robot description, xacro)
@@ -24,5 +24,5 @@
     <!-- D435 camera -->
     <xacro:property name="camera_pose_file"
-                    value="$(find panda_torque_mpc)/franka/manipulation/config/calibrated-params.yaml" />
+                    value="$(find panda_torque_mpc)/config/calibrated-params.yaml" />
     <xacro:property name="camera_pose" value="${load_yaml(camera_pose_file)}"/>
     <link name="${arm_id}_ref_camera_link"/>
@@ -51,5 +51,5 @@
         <origin xyz="0.022 0 -0.012" rpy="3.141592653589793 0 -1.5707963267948966"/>
         <geometry>
-          <mesh filename="package://agimus_demos/franka/manipulation/meshes/camera-support.stl" scale="1 1 1"/>
+          <mesh filename="package://panda_torque_mpc/meshes/camera-support.stl" scale="1 1 1"/>
         </geometry>
       </visual>
@@ -57,5 +57,5 @@
         <origin xyz="0.022 0 -0.012" rpy="3.141592653589793 0 -1.5707963267948966"/>
         <geometry>
-          <mesh filename="package://agimus_demos/franka/manipulation/meshes/camera-support.stl" scale="1 1 1"/>
+          <mesh filename="package://panda_torque_mpc/meshes/camera-support.stl" scale="1 1 1"/>
         </geometry>
       </collision>

Commit message: Merging debug branch to main (#11)
* Change pinocchio version

* Change hardcoded paths in favour of ROS packages

* Fix pinocchio not finding mesh paths

* Fix getters issue

* Add abiulity to disable camera | update compilation flags

* Reduce number of build flags in readme

* Add disabling camera to the README file

* Change goal poses for the pose publisher

* Fix MPC controller initialization | remove unuzed collision

* deleting post treatment and putting it in separate repo (#10)

Co-authored-by: Arthur <arthur.haffemayer@laas.fr>

---------

Co-authored-by: Krzysztof Wojciechowski <krzy.wojciecho@gmail.com>
Co-authored-by: Arthur <arthur.haffemayer@laas.fr>

File: urdf/franka_robot.xacro (robot description, xacro)
@@ -9,4 +9,5 @@
     <!-- Is the robot being simulated in gazebo?" -->
     <xacro:arg name="gazebo" default="false" />
+    <xacro:arg name="simulate_camera" default="false" />
     <xacro:include filename="$(find panda_torque_mpc)/urdf/utils.xacro" />
     <xacro:include filename="$(find panda_torque_mpc)/urdf/franka_arm.xacro" />
@@ -66,5 +67,7 @@
       <origin xyz="0 0 0" rpy="3.141592653589793 0 0"/>
     </joint>
-    <xacro:if value="$(arg gazebo)">
+    <xacro:property name="gz_on" value="$(arg gazebo)" />
+    <xacro:property name="sim_cam_on" value="$(arg simulate_camera)" />
+    <xacro:if value="${gz_on and sim_cam_on}">
       <xacro:include filename="$(find panda_torque_mpc)/urdf/_d435.gazebo.xacro"/>
       <xacro:gazebo_d435 camera_name="d435"
