Commit message: python node warm start working

File: urdf/support.urdf.xacro (robot description, xacro)
@@ -54,5 +54,5 @@
           <origin xyz="0 0 0"/>
           <geometry>
-            <sphere radius="0.15"/>
+            <sphere radius="0.1"/>
           </geometry>
           <material name="green">
@@ -63,5 +63,5 @@
           <origin xyz="0 0 0"/>
           <geometry>
-            <sphere radius="0.15"/>
+            <sphere radius="0.1"/>
           </geometry>
         </collision>

Commit message: getting rid of the warmstart remains

File: urdf/support.urdf.xacro (robot description, xacro)
@@ -54,5 +54,5 @@
           <origin xyz="0 0 0"/>
           <geometry>
-            <sphere radius="0.1"/>
+            <sphere radius="0.15"/>
           </geometry>
           <material name="green">
@@ -63,5 +63,5 @@
           <origin xyz="0 0 0"/>
           <geometry>
-            <sphere radius="0.1"/>
+            <sphere radius="0.15"/>
           </geometry>
         </collision>

Commit message: Feature/add visualization obstacle (#18)
* URDF Generator class

* adding capsule in urdf parser

* visualizer, but the markers aren't detected

* obstacle found in yaml

* works on rviz

* adding to gazebo, model is printed but not plotted

* yaml to gazebo works but the obstacle isn't avoided

* updating cmake list & readme

* fixing colors

* works for the sphere but not the cylinder and the box

* simplify the sdf str. Still doesn't work with cylinder & box

* visualization works but not the collision avoidance yet

* working for all obstacles

* taking capsules into consideration

* reducing collision model (error of shared pointer)

* reducing collision model

* final exp running on sim

* working setup for exp

* experiment box avoiding working

* delete comments

* Update include/panda_torque_mpc/reduce_collision_model.h

Co-authored-by: Krzysztof Wojciechowski <49921081+Kotochleb@users.noreply.github.com>

* undoing formatter changes

* comment on hardcoding reduce collision model

* Update include/panda_torque_mpc/reduce_collision_model.h

Co-authored-by: Krzysztof Wojciechowski <49921081+Kotochleb@users.noreply.github.com>

* Update include/panda_torque_mpc/reduce_collision_model.h

Co-authored-by: Krzysztof Wojciechowski <49921081+Kotochleb@users.noreply.github.com>

* Update include/panda_torque_mpc/reduce_collision_model.h

Co-authored-by: Krzysztof Wojciechowski <49921081+Kotochleb@users.noreply.github.com>

* Update include/panda_torque_mpc/reduce_collision_model.h

Co-authored-by: Krzysztof Wojciechowski <49921081+Kotochleb@users.noreply.github.com>

* Update include/panda_torque_mpc/reduce_collision_model.h

Co-authored-by: Krzysztof Wojciechowski <49921081+Kotochleb@users.noreply.github.com>

* Update nodes/obstacle_visualizer.py

Co-authored-by: Krzysztof Wojciechowski <49921081+Kotochleb@users.noreply.github.com>

* Update nodes/obstacle_visualizer.py

Co-authored-by: Krzysztof Wojciechowski <49921081+Kotochleb@users.noreply.github.com>

* Update nodes/obstacle_visualizer.py

Co-authored-by: Krzysztof Wojciechowski <49921081+Kotochleb@users.noreply.github.com>

* Update nodes/obstacle_visualizer.py

Co-authored-by: Krzysztof Wojciechowski <49921081+Kotochleb@users.noreply.github.com>

* Update nodes/obstacle_visualizer.py

Co-authored-by: Krzysztof Wojciechowski <49921081+Kotochleb@users.noreply.github.com>

* adding docstrings

* correcting deleted lines by auto commit from suggestion

* commenting the magic of urdf

* adding a rosparam for the visualization of the obstacles

* type hinting

* type hinting v2

* indentation

---------

Co-authored-by: Arthur Haffemayer <ahaffemaye@miyanoura>
Co-authored-by: Krzysztof Wojciechowski <49921081+Kotochleb@users.noreply.github.com>

File: urdf/support.urdf.xacro (robot description, xacro)
@@ -44,26 +44,4 @@
           </geometry>
         </collision> -->
-      </link>
-      <link name="the_ball">
-        <inertial>
-          <mass value="1"/>
-          <origin xyz="0 0 0"/>
-          <inertia ixx="1"  ixy="0"  ixz="0" iyy="1" iyz="0" izz="1" />
-        </inertial>
-        <visual>
-          <origin xyz="0 0 0"/>
-          <geometry>
-            <sphere radius="0.15"/>
-          </geometry>
-          <material name="green">
-            <color rgba ="0 1 0 0.8"/>
-          </material>
-        </visual>
-        <collision>
-          <origin xyz="0 0 0"/>
-          <geometry>
-            <sphere radius="0.15"/>
-          </geometry>
-        </collision>
       </link>
       <link name="wall_link_1">
@@ -206,9 +184,4 @@
         <child link="panda1_box"/>
       </joint>
-      <joint name="the_ball_joint" type="fixed">
-        <origin xyz="0 0 0.8" />
-        <parent link="world"/>
-        <child link="the_ball"/>
-      </joint>
   </xacro:macro>
 </robot>
