Commit message: Obtain rosbot.urdf with xacro without manual changes

File: urdf/franka_arm.xacro (robot description, xacro)
@@ -5,5 +5,5 @@
   <!-- arm_id: Namespace of the robot arm. Serves to differentiate between arms in case of multiple instances. -->
   <!-- joint_limits: description of the joint limits that comes from a YAML file. Example definition: ${xacro.load_yaml('$(find franka_description)/robots/fr3/joint_limits.yaml')} -->
-  <xacro:macro name="franka_arm" params="arm_id:='panda' description_pkg:='franka_description' connected_to:='' xyz:='0 0 0' rpy:='0 0 0' gazebo:=false safety_distance:=0 joint_limits" >
+  <xacro:macro name="franka_arm" params="arm_id:='panda' description_pkg:='franka_description' connected_to:='' xyz:='0 0 0' rpy:='0 0 0' gazebo:=false pinocchio_colisions:=false safety_distance:=0 joint_limits" >
     <xacro:unless value="${not connected_to}">
       <joint name="${arm_id}_joint_${connected_to}" type="fixed">
@@ -13,10 +13,10 @@
       </joint>
     </xacro:unless>
-    <xacro:link_with_sc name="link0" gazebo="${gazebo}">
+    <xacro:link_with_sc name="link0" gazebo="${gazebo}" pinocchio_colisions="${pinocchio_colisions}">
       <self_collision_geometries>
         <xacro:collision_capsule xyz="-0.075 0 0.06" direction="x" radius="${0.06+safety_distance}" length="0.03" />
       </self_collision_geometries>
     </xacro:link_with_sc>
-    <xacro:link_with_sc name="link1" gazebo="${gazebo}">
+    <xacro:link_with_sc name="link1" gazebo="${gazebo}" pinocchio_colisions="${pinocchio_colisions}">
       <self_collision_geometries>
         <xacro:collision_capsule xyz="0 0 -191.5e-3" radius="${0.06+safety_distance}" length="0.283" />
@@ -31,5 +31,5 @@
       <dynamics D="1" K="7000" damping="0.003" friction="0.0" mu_coulomb="0" mu_viscous="16" />
     </joint>
-    <xacro:link_with_sc name="link2" gazebo="${gazebo}">
+    <xacro:link_with_sc name="link2" gazebo="${gazebo}" pinocchio_colisions="${pinocchio_colisions}">
       <self_collision_geometries>
         <xacro:collision_capsule xyz="0 0 0" radius="${0.06+safety_distance}" length="0.12" />
@@ -44,5 +44,5 @@
       <dynamics D="1" K="7000" damping="0.003" friction="0.0" mu_coulomb="0" mu_viscous="16" />
     </joint>
-    <xacro:link_with_sc name="link3" gazebo="${gazebo}">
+    <xacro:link_with_sc name="link3" gazebo="${gazebo}" pinocchio_colisions="${pinocchio_colisions}">
       <self_collision_geometries>
         <xacro:collision_capsule xyz="0 0 -0.145" radius="${0.06+safety_distance}" length="0.15" />
@@ -57,5 +57,5 @@
       <dynamics D="1" K="7000" damping="0.003" friction="0.0" mu_coulomb="0" mu_viscous="16" />
     </joint>
-    <xacro:link_with_sc name="link4" gazebo="${gazebo}">
+    <xacro:link_with_sc name="link4" gazebo="${gazebo}" pinocchio_colisions="${pinocchio_colisions}">
       <self_collision_geometries>
         <xacro:collision_capsule xyz="0 0 0" radius="${0.06+safety_distance}" length="0.12" />
@@ -70,5 +70,5 @@
       <dynamics D="1" K="7000" damping="0.003" friction="0.0" mu_coulomb="0" mu_viscous="16" />
     </joint>
-    <xacro:link_with_sc name="link5" gazebo="${gazebo}">
+    <xacro:link_with_sc name="link5" gazebo="${gazebo}" pinocchio_colisions="${pinocchio_colisions}">
       <self_collision_geometries>
         <xacro:collision_capsule xyz="0 0 -0.26"    radius="${0.060+safety_distance}" length="0.10" />
@@ -84,5 +84,5 @@
       <dynamics D="1" K="7000" damping="0.003" friction="0.0" mu_coulomb="0" mu_viscous="16" />
     </joint>
-    <xacro:link_with_sc name="link6" gazebo="${gazebo}">
+    <xacro:link_with_sc name="link6" gazebo="${gazebo}" pinocchio_colisions="${pinocchio_colisions}">
       <self_collision_geometries>
         <xacro:collision_capsule xyz="0 0 -0.03" radius="${0.05+safety_distance}" length="0.08" />
@@ -97,5 +97,5 @@
       <dynamics D="1" K="7000" damping="0.003" friction="0.0" mu_coulomb="0" mu_viscous="16" />
     </joint>
-    <xacro:link_with_sc name="link7" gazebo="${gazebo}" rpy="0 0 ${pi/4}">
+    <xacro:link_with_sc name="link7" gazebo="${gazebo}" pinocchio_colisions="${pinocchio_colisions}" rpy="0 0 ${pi/4}">
       <self_collision_geometries>
         <xacro:collision_capsule xyz="0 0 0.01" direction="z" radius="${0.04+safety_distance}" length="0.14" />
@@ -111,5 +111,11 @@
       <dynamics D="1" K="7000" damping="0.003" friction="0.0" mu_coulomb="0" mu_viscous="16"/>
     </joint>
-    <link name="${arm_id}_link8"/>
+    <link name="${arm_id}_link8">
+      <inertial>
+        <mass value="0"/>
+        <origin rpy="0 0 0" xyz="0 0 0"/>
+        <inertia ixx="0" ixy="0" ixz="0" iyy="0" iyz="0" izz="0"/>
+      </inertial>
+    </link>
     <joint name="${arm_id}_joint8" type="fixed">
       <origin rpy="0 0 0" xyz="0 0 0.107"/>

File: urdf/franka_hand.xacro (robot description, xacro)
@@ -2,5 +2,5 @@
 <robot xmlns:xacro="http://www.ros.org/wiki/xacro" name="hand">
   <!-- safety_distance: Minimum safety distance in [m] by which the collision volumes are expanded and which is enforced during robot motions -->
-  <xacro:macro name="franka_hand" params="connected_to:='' arm_id rpy:='0 0 0' xyz:='0 0 0' tcp_xyz:='0 0 0.1034' tcp_rpy:='0 0 0' safety_distance:=0 gazebo:=false description_pkg:=franka_description">
+  <xacro:macro name="franka_hand" params="connected_to:='' arm_id rpy:='0 0 0' xyz:='0 0 0' tcp_xyz:='0 0 0.1034' tcp_rpy:='0 0 0' safety_distance:=0 gazebo:=false pinocchio_colisions:=false description_pkg:=franka_description">
     <xacro:unless value="${connected_to == ''}">
       <joint name="${arm_id}_hand_joint" type="fixed">
@@ -15,5 +15,11 @@
     </xacro:link_with_sc>
     <!-- Define the hand_tcp frame -->
-    <link name="${arm_id}_hand_tcp" />
+    <link name="${arm_id}_hand_tcp">
+      <inertial>
+        <mass value="0"/>
+        <origin rpy="0 0 0" xyz="0 0 0"/>
+        <inertia ixx="0" ixy="0" ixz="0" iyy="0" iyz="0" izz="0"/>
+      </inertial>
+    </link>
     <joint name="${arm_id}_hand_tcp_joint" type="fixed">
       <origin xyz="${tcp_xyz}" rpy="${tcp_rpy}" />
@@ -27,14 +33,40 @@
         </geometry>
       </visual>
-      <!-- approx sphere -->
+      <!-- screw mount -->
       <collision>
-        <origin rpy="0 0 0" xyz="0 18.5e-3 11e-3"/>
+        <origin xyz="0 18.5e-3 11e-3" rpy="0 0 0" />
         <geometry>
-          <sphere radius=".03"/>
+          <xacro:if value="${pinocchio_colisions}">
+            <sphere radius=".03"/>
+          </xacro:if>
+          <xacro:unless value="${pinocchio_colisions}">
+            <box size="22e-3 15e-3 20e-3" />
+          </xacro:unless>
         </geometry>
       </collision>
-      <xacro:if value="${gazebo}">
-        <xacro:inertial_props name="leftfinger" />
-      </xacro:if>
+      <xacro:unless value="${pinocchio_colisions}">
+        <!-- cartriage sledge -->
+        <collision>
+          <origin xyz="0 6.8e-3 2.2e-3" rpy="0 0 0" />
+          <geometry>
+            <box size="22e-3 8.8e-3 3.8e-3" />
+          </geometry>
+        </collision>
+        <!-- diagonal finger -->
+        <collision>
+          <origin xyz="0 15.9e-3 28.35e-3" rpy="${pi/6} 0 0" />
+          <geometry>
+            <box size="17.5e-3 7e-3 23.5e-3" />
+          </geometry>
+        </collision>
+        <!-- rubber tip with which to grasp -->
+        <collision>
+          <origin xyz="0 7.58e-3 45.25e-3" rpy="0 0 0" />
+          <geometry>
+            <box size="17.5e-3 15.2e-3 18.5e-3" />
+          </geometry>
+        </collision>
+      </xacro:unless>
+      <xacro:inertial_props name="leftfinger" />
     </link>
     <link name="${arm_id}_rightfinger">
@@ -45,14 +77,40 @@
         </geometry>
       </visual>
-      <!-- approx sphere -->
+      <!-- screw mount -->
       <collision>
-        <origin rpy="0 0 0" xyz="0 -18.5e-3 11e-3"/>
+        <origin xyz="0 -18.5e-3 11e-3" rpy="0 0 0" />
         <geometry>
-          <sphere radius=".03"/>
+          <xacro:if value="${pinocchio_colisions}">
+            <sphere radius=".03"/>
+          </xacro:if>
+          <xacro:unless value="${pinocchio_colisions}">
+            <box size="22e-3 15e-3 20e-3" />
+          </xacro:unless>
         </geometry>
       </collision>
-      <xacro:if value="${gazebo}">
-        <xacro:inertial_props name="rightfinger" />
-      </xacro:if>
+      <xacro:unless value="${pinocchio_colisions}">
+      <!-- cartriage sledge -->
+      <collision>
+        <origin xyz="0 -6.8e-3 2.2e-3" rpy="0 0 0" />
+        <geometry>
+          <box size="22e-3 8.8e-3 3.8e-3" />
+        </geometry>
+      </collision>
+      <!-- diagonal finger -->
+      <collision>
+        <origin xyz="0 -15.9e-3 28.35e-3" rpy="${-pi/6} 0 0" />
+        <geometry>
+          <box size="17.5e-3 7e-3 23.5e-3" />
+        </geometry>
+      </collision>
+      <!-- rubber tip with which to grasp -->
+      <collision>
+        <origin xyz="0 -7.58e-3 45.25e-3" rpy="0 0 0" />
+        <geometry>
+          <box size="17.5e-3 15.2e-3 18.5e-3" />
+        </geometry>
+        </collision>
+      </xacro:unless>
+      <xacro:inertial_props name="rightfinger" />
     </link>
     <joint name="${arm_id}_finger_joint1" type="prismatic">

File: urdf/franka_robot.xacro (robot description, xacro)
@@ -9,9 +9,14 @@
     <!-- Is the robot being simulated in gazebo?" -->
     <xacro:arg name="gazebo" default="false" />
+    <xacro:arg name="pinocchio_colisions" default="false" />
     <xacro:arg name="simulate_camera" default="false" />
     <xacro:include filename="$(find panda_torque_mpc)/urdf/utils.xacro" />
     <xacro:include filename="$(find panda_torque_mpc)/urdf/franka_arm.xacro" />
     <xacro:include filename="$(find panda_torque_mpc)/urdf/franka_hand.xacro"/>
-    <xacro:franka_arm arm_id="${arm_id}" safety_distance="0.03" gazebo="$(arg gazebo)" joint_limits="${joint_limits}"/>
+    <xacro:franka_arm arm_id="${arm_id}"
+                      safety_distance="0.03"
+                      gazebo="$(arg gazebo)"
+                      pinocchio_colisions="$(arg pinocchio_colisions)"
+                      joint_limits="${joint_limits}"/>
     <xacro:franka_hand
         arm_id="${arm_id}"
@@ -22,4 +27,5 @@
         safety_distance="0.03"
         gazebo="$(arg gazebo)"
+        pinocchio_colisions="$(arg pinocchio_colisions)"
         />
     <!-- D435 camera -->

File: urdf/support.urdf.xacro (robot description, xacro)
@@ -2,4 +2,5 @@
 <robot xmlns:xacro="http://www.ros.org/wiki/xacro">
   <xacro:macro name="support" params="">
+      <xacro:arg name="pinocchio_colisions" default="false" />
       <link name="support_link">
         <inertial>
@@ -14,10 +15,12 @@
           </geometry>
         </visual>
-        <!-- <collision>
-          <origin xyz="0 0 0.38"/>
-          <geometry>
-	    <box size="1.703 0.803 0.76"/>
-          </geometry>
-        </collision> -->
+        <xacro:if value="$(arg pinocchio_colisions)">
+          <collision>
+            <origin xyz="0 0 0.38"/>
+            <geometry>
+        <box size="1.703 0.803 0.76"/>
+            </geometry>
+          </collision>
+        </xacro:if>
         <!--visual>
           <origin xyz="-0.61 0.2215 0.77"/>
@@ -38,10 +41,12 @@
           </geometry>
         </visual>
-        <!-- <collision>
-          <origin xyz="0.6385 -0.1655 0.77"/>
-          <geometry>
-            <box size="0.3 0.3 0.02"/>
-          </geometry>
-        </collision> -->
+        <xacro:if value="$(arg pinocchio_colisions)">
+          <collision>
+            <origin xyz="0.6385 -0.1655 0.77"/>
+            <geometry>
+              <box size="0.3 0.3 0.02"/>
+            </geometry>
+          </collision>
+        </xacro:if>
       </link>
       <link name="wall_link_1">
@@ -184,4 +189,28 @@
         <child link="panda1_box"/>
       </joint>
+      <gazebo reference="support_link">
+        <static>true</static>
+        <kinematic>false</kinematic>
+      </gazebo>
+      <gazebo reference="wall_link_1">
+        <static>true</static>
+        <kinematic>false</kinematic>
+      </gazebo>
+      <gazebo reference="wall_link_2">
+        <static>true</static>
+        <kinematic>false</kinematic>
+      </gazebo>
+      <gazebo reference="wall_link_3">
+        <static>true</static>
+        <kinematic>false</kinematic>
+      </gazebo>
+      <gazebo reference="pedestal">
+        <static>true</static>
+        <kinematic>false</kinematic>
+      </gazebo>
+      <gazebo reference="panda1_box">
+        <static>true</static>
+        <kinematic>false</kinematic>
+      </gazebo>
   </xacro:macro>
 </robot>

File: urdf/utils.xacro (robot description, xacro)
@@ -33,5 +33,5 @@
   <!-- self_collision_geometries:  self <collision> models        -->
   <!-- ========================================================== -->
-  <xacro:macro name="link_with_sc" params="name prefix=${arm_id}_ rpy:='0 0 0' **self_collision_geometries gazebo:=false">
+  <xacro:macro name="link_with_sc" params="name prefix=${arm_id}_ rpy:='0 0 0' **self_collision_geometries gazebo:=false pinocchio_colisions:=false">
     <!-- sub-link defining detailed meshes for collision with environment -->
     <link name="${prefix}${name}">
@@ -43,15 +43,15 @@
       <collision>
         <geometry>
-          <mesh filename="package://franka_description/meshes/collision/${name}.stl" />
+          <mesh filename="package://${description_pkg}/meshes/collision/${name}.stl" />
         </geometry>
       </collision>
-      <xacro:if value="${gazebo}">
-        <xacro:inertial_props name="${name}" />
-      </xacro:if>
+      <xacro:inertial_props name="${name}" />
     </link>
     <!-- sub-link defining coarse geometries of real robot's internal self-collision -->
     <link name="${prefix}${name}_sc">
       <xacro:unless value="${gazebo}">
-        <xacro:insert_block name="self_collision_geometries" />
+        <xacro:if value="${pinocchio_colisions}">
+          <xacro:insert_block name="self_collision_geometries" />
+        </xacro:if>
       </xacro:unless>
     </link>
