Commit message: Fix `pinocchio_colisions` typo

File: urdf/franka_arm.xacro (robot description, xacro)
@@ -5,5 +5,5 @@
   <!-- arm_id: Namespace of the robot arm. Serves to differentiate between arms in case of multiple instances. -->
   <!-- joint_limits: description of the joint limits that comes from a YAML file. Example definition: ${xacro.load_yaml('$(find franka_description)/robots/fr3/joint_limits.yaml')} -->
-  <xacro:macro name="franka_arm" params="arm_id:='panda' description_pkg:='franka_description' connected_to:='' xyz:='0 0 0' rpy:='0 0 0' gazebo:=false pinocchio_colisions:=false safety_distance:=0 joint_limits" >
+  <xacro:macro name="franka_arm" params="arm_id:='panda' description_pkg:='franka_description' connected_to:='' xyz:='0 0 0' rpy:='0 0 0' gazebo:=false pinocchio_collisions:=false safety_distance:=0 joint_limits" >
     <xacro:unless value="${not connected_to}">
       <joint name="${arm_id}_joint_${connected_to}" type="fixed">
@@ -13,10 +13,10 @@
       </joint>
     </xacro:unless>
-    <xacro:link_with_sc name="link0" gazebo="${gazebo}" pinocchio_colisions="${pinocchio_colisions}">
+    <xacro:link_with_sc name="link0" gazebo="${gazebo}" pinocchio_collisions="${pinocchio_collisions}">
       <self_collision_geometries>
         <xacro:collision_capsule xyz="-0.075 0 0.06" direction="x" radius="${0.06+safety_distance}" length="0.03" />
       </self_collision_geometries>
     </xacro:link_with_sc>
-    <xacro:link_with_sc name="link1" gazebo="${gazebo}" pinocchio_colisions="${pinocchio_colisions}">
+    <xacro:link_with_sc name="link1" gazebo="${gazebo}" pinocchio_collisions="${pinocchio_collisions}">
       <self_collision_geometries>
         <xacro:collision_capsule xyz="0 0 -191.5e-3" radius="${0.06+safety_distance}" length="0.283" />
@@ -31,5 +31,5 @@
       <dynamics D="1" K="7000" damping="0.003" friction="0.0" mu_coulomb="0" mu_viscous="16" />
     </joint>
-    <xacro:link_with_sc name="link2" gazebo="${gazebo}" pinocchio_colisions="${pinocchio_colisions}">
+    <xacro:link_with_sc name="link2" gazebo="${gazebo}" pinocchio_collisions="${pinocchio_collisions}">
       <self_collision_geometries>
         <xacro:collision_capsule xyz="0 0 0" radius="${0.06+safety_distance}" length="0.12" />
@@ -44,5 +44,5 @@
       <dynamics D="1" K="7000" damping="0.003" friction="0.0" mu_coulomb="0" mu_viscous="16" />
     </joint>
-    <xacro:link_with_sc name="link3" gazebo="${gazebo}" pinocchio_colisions="${pinocchio_colisions}">
+    <xacro:link_with_sc name="link3" gazebo="${gazebo}" pinocchio_collisions="${pinocchio_collisions}">
       <self_collision_geometries>
         <xacro:collision_capsule xyz="0 0 -0.145" radius="${0.06+safety_distance}" length="0.15" />
@@ -57,5 +57,5 @@
       <dynamics D="1" K="7000" damping="0.003" friction="0.0" mu_coulomb="0" mu_viscous="16" />
     </joint>
-    <xacro:link_with_sc name="link4" gazebo="${gazebo}" pinocchio_colisions="${pinocchio_colisions}">
+    <xacro:link_with_sc name="link4" gazebo="${gazebo}" pinocchio_collisions="${pinocchio_collisions}">
       <self_collision_geometries>
         <xacro:collision_capsule xyz="0 0 0" radius="${0.06+safety_distance}" length="0.12" />
@@ -70,5 +70,5 @@
       <dynamics D="1" K="7000" damping="0.003" friction="0.0" mu_coulomb="0" mu_viscous="16" />
     </joint>
-    <xacro:link_with_sc name="link5" gazebo="${gazebo}" pinocchio_colisions="${pinocchio_colisions}">
+    <xacro:link_with_sc name="link5" gazebo="${gazebo}" pinocchio_collisions="${pinocchio_collisions}">
       <self_collision_geometries>
         <xacro:collision_capsule xyz="0 0 -0.26"    radius="${0.060+safety_distance}" length="0.10" />
@@ -84,5 +84,5 @@
       <dynamics D="1" K="7000" damping="0.003" friction="0.0" mu_coulomb="0" mu_viscous="16" />
     </joint>
-    <xacro:link_with_sc name="link6" gazebo="${gazebo}" pinocchio_colisions="${pinocchio_colisions}">
+    <xacro:link_with_sc name="link6" gazebo="${gazebo}" pinocchio_collisions="${pinocchio_collisions}">
       <self_collision_geometries>
         <xacro:collision_capsule xyz="0 0 -0.03" radius="${0.05+safety_distance}" length="0.08" />
@@ -97,5 +97,5 @@
       <dynamics D="1" K="7000" damping="0.003" friction="0.0" mu_coulomb="0" mu_viscous="16" />
     </joint>
-    <xacro:link_with_sc name="link7" gazebo="${gazebo}" pinocchio_colisions="${pinocchio_colisions}" rpy="0 0 ${pi/4}">
+    <xacro:link_with_sc name="link7" gazebo="${gazebo}" pinocchio_collisions="${pinocchio_collisions}" rpy="0 0 ${pi/4}">
       <self_collision_geometries>
         <xacro:collision_capsule xyz="0 0 0.01" direction="z" radius="${0.04+safety_distance}" length="0.14" />

File: urdf/franka_hand.xacro (robot description, xacro)
@@ -2,5 +2,5 @@
 <robot xmlns:xacro="http://www.ros.org/wiki/xacro" name="hand">
   <!-- safety_distance: Minimum safety distance in [m] by which the collision volumes are expanded and which is enforced during robot motions -->
-  <xacro:macro name="franka_hand" params="connected_to:='' arm_id rpy:='0 0 0' xyz:='0 0 0' tcp_xyz:='0 0 0.1034' tcp_rpy:='0 0 0' safety_distance:=0 gazebo:=false pinocchio_colisions:=false description_pkg:=franka_description">
+  <xacro:macro name="franka_hand" params="connected_to:='' arm_id rpy:='0 0 0' xyz:='0 0 0' tcp_xyz:='0 0 0.1034' tcp_rpy:='0 0 0' safety_distance:=0 gazebo:=false pinocchio_collisions:=false description_pkg:=franka_description">
     <xacro:unless value="${connected_to == ''}">
       <joint name="${arm_id}_hand_joint" type="fixed">
@@ -37,13 +37,13 @@
         <origin xyz="0 18.5e-3 11e-3" rpy="0 0 0" />
         <geometry>
-          <xacro:if value="${pinocchio_colisions}">
+          <xacro:if value="${pinocchio_collisions}">
             <sphere radius=".03"/>
           </xacro:if>
-          <xacro:unless value="${pinocchio_colisions}">
+          <xacro:unless value="${pinocchio_collisions}">
             <box size="22e-3 15e-3 20e-3" />
           </xacro:unless>
         </geometry>
       </collision>
-      <xacro:unless value="${pinocchio_colisions}">
+      <xacro:unless value="${pinocchio_collisions}">
         <!-- cartriage sledge -->
         <collision>
@@ -81,13 +81,13 @@
         <origin xyz="0 -18.5e-3 11e-3" rpy="0 0 0" />
         <geometry>
-          <xacro:if value="${pinocchio_colisions}">
+          <xacro:if value="${pinocchio_collisions}">
             <sphere radius=".03"/>
           </xacro:if>
-          <xacro:unless value="${pinocchio_colisions}">
+          <xacro:unless value="${pinocchio_collisions}">
             <box size="22e-3 15e-3 20e-3" />
           </xacro:unless>
         </geometry>
       </collision>
-      <xacro:unless value="${pinocchio_colisions}">
+      <xacro:unless value="${pinocchio_collisions}">
       <!-- cartriage sledge -->
       <collision>

File: urdf/franka_robot.xacro (robot description, xacro)
@@ -9,5 +9,5 @@
     <!-- Is the robot being simulated in gazebo?" -->
     <xacro:arg name="gazebo" default="false" />
-    <xacro:arg name="pinocchio_colisions" default="false" />
+    <xacro:arg name="pinocchio_collisions" default="false" />
     <xacro:arg name="simulate_camera" default="false" />
     <xacro:include filename="$(find panda_torque_mpc)/urdf/utils.xacro" />
@@ -17,5 +17,5 @@
                       safety_distance="0.03"
                       gazebo="$(arg gazebo)"
-                      pinocchio_colisions="$(arg pinocchio_colisions)"
+                      pinocchio_collisions="$(arg pinocchio_collisions)"
                       joint_limits="${joint_limits}"/>
     <xacro:franka_hand
@@ -27,5 +27,5 @@
         safety_distance="0.03"
         gazebo="$(arg gazebo)"
-        pinocchio_colisions="$(arg pinocchio_colisions)"
+        pinocchio_collisions="$(arg pinocchio_collisions)"
         />
     <!-- D435 camera -->

File: urdf/support.urdf.xacro (robot description, xacro)
@@ -2,5 +2,5 @@
 <robot xmlns:xacro="http://www.ros.org/wiki/xacro">
   <xacro:macro name="support" params="">
-      <xacro:arg name="pinocchio_colisions" default="false" />
+      <xacro:arg name="pinocchio_collisions" default="false" />
       <link name="support_link">
         <inertial>
@@ -15,5 +15,5 @@
           </geometry>
         </visual>
-        <xacro:if value="$(arg pinocchio_colisions)">
+        <xacro:if value="$(arg pinocchio_collisions)">
           <collision>
             <origin xyz="0 0 0.38"/>
@@ -41,5 +41,5 @@
           </geometry>
         </visual>
-        <xacro:if value="$(arg pinocchio_colisions)">
+        <xacro:if value="$(arg pinocchio_collisions)">
           <collision>
             <origin xyz="0.6385 -0.1655 0.77"/>

File: urdf/utils.xacro (robot description, xacro)
@@ -33,5 +33,5 @@
   <!-- self_collision_geometries:  self <collision> models        -->
   <!-- ========================================================== -->
-  <xacro:macro name="link_with_sc" params="name prefix=${arm_id}_ rpy:='0 0 0' **self_collision_geometries gazebo:=false pinocchio_colisions:=false">
+  <xacro:macro name="link_with_sc" params="name prefix=${arm_id}_ rpy:='0 0 0' **self_collision_geometries gazebo:=false pinocchio_collisions:=false">
     <!-- sub-link defining detailed meshes for collision with environment -->
     <link name="${prefix}${name}">
@@ -51,5 +51,5 @@
     <link name="${prefix}${name}_sc">
       <xacro:unless value="${gazebo}">
-        <xacro:if value="${pinocchio_colisions}">
+        <xacro:if value="${pinocchio_collisions}">
           <xacro:insert_block name="self_collision_geometries" />
         </xacro:if>
