Commit message: Use single URDF for both Pinocchio and ROS

File: urdf/franka_hand.xacro (robot description, xacro)
@@ -27,30 +27,9 @@
         </geometry>
       </visual>
-      <!-- screw mount -->
+      <!-- approx sphere -->
       <collision>
-        <origin xyz="0 18.5e-3 11e-3" rpy="0 0 0" />
+        <origin rpy="0 0 0" xyz="0 18.5e-3 11e-3"/>
         <geometry>
-          <box size="22e-3 15e-3 20e-3" />
-        </geometry>
-      </collision>
-      <!-- cartriage sledge -->
-      <collision>
-        <origin xyz="0 6.8e-3 2.2e-3" rpy="0 0 0" />
-        <geometry>
-          <box size="22e-3 8.8e-3 3.8e-3" />
-        </geometry>
-      </collision>
-      <!-- diagonal finger -->
-      <collision>
-        <origin xyz="0 15.9e-3 28.35e-3" rpy="${pi/6} 0 0" />
-        <geometry>
-          <box size="17.5e-3 7e-3 23.5e-3" />
-        </geometry>
-      </collision>
-      <!-- rubber tip with which to grasp -->
-      <collision>
-        <origin xyz="0 7.58e-3 45.25e-3" rpy="0 0 0" />
-        <geometry>
-          <box size="17.5e-3 15.2e-3 18.5e-3" />
+          <sphere radius=".03"/>
         </geometry>
       </collision>
@@ -66,30 +45,9 @@
         </geometry>
       </visual>
-      <!-- screw mount -->
+      <!-- approx sphere -->
       <collision>
-        <origin xyz="0 -18.5e-3 11e-3" rpy="0 0 0" />
+        <origin rpy="0 0 0" xyz="0 -18.5e-3 11e-3"/>
         <geometry>
-          <box size="22e-3 15e-3 20e-3" />
-        </geometry>
-      </collision>
-      <!-- cartriage sledge -->
-      <collision>
-        <origin xyz="0 -6.8e-3 2.2e-3" rpy="0 0 0" />
-        <geometry>
-          <box size="22e-3 8.8e-3 3.8e-3" />
-        </geometry>
-      </collision>
-      <!-- diagonal finger -->
-      <collision>
-        <origin xyz="0 -15.9e-3 28.35e-3" rpy="${-pi/6} 0 0" />
-        <geometry>
-          <box size="17.5e-3 7e-3 23.5e-3" />
-        </geometry>
-      </collision>
-      <!-- rubber tip with which to grasp -->
-      <collision>
-        <origin xyz="0 -7.58e-3 45.25e-3" rpy="0 0 0" />
-        <geometry>
-          <box size="17.5e-3 15.2e-3 18.5e-3" />
+          <sphere radius=".03"/>
         </geometry>
       </collision>

Commit message: Revert "Use single URDF for both Pinocchio and ROS"

File: urdf/franka_hand.xacro (robot description, xacro)
@@ -27,9 +27,30 @@
         </geometry>
       </visual>
-      <!-- approx sphere -->
+      <!-- screw mount -->
       <collision>
-        <origin rpy="0 0 0" xyz="0 18.5e-3 11e-3"/>
+        <origin xyz="0 18.5e-3 11e-3" rpy="0 0 0" />
         <geometry>
-          <sphere radius=".03"/>
+          <box size="22e-3 15e-3 20e-3" />
+        </geometry>
+      </collision>
+      <!-- cartriage sledge -->
+      <collision>
+        <origin xyz="0 6.8e-3 2.2e-3" rpy="0 0 0" />
+        <geometry>
+          <box size="22e-3 8.8e-3 3.8e-3" />
+        </geometry>
+      </collision>
+      <!-- diagonal finger -->
+      <collision>
+        <origin xyz="0 15.9e-3 28.35e-3" rpy="${pi/6} 0 0" />
+        <geometry>
+          <box size="17.5e-3 7e-3 23.5e-3" />
+        </geometry>
+      </collision>
+      <!-- rubber tip with which to grasp -->
+      <collision>
+        <origin xyz="0 7.58e-3 45.25e-3" rpy="0 0 0" />
+        <geometry>
+          <box size="17.5e-3 15.2e-3 18.5e-3" />
         </geometry>
       </collision>
@@ -45,9 +66,30 @@
         </geometry>
       </visual>
-      <!-- approx sphere -->
+      <!-- screw mount -->
       <collision>
-        <origin rpy="0 0 0" xyz="0 -18.5e-3 11e-3"/>
+        <origin xyz="0 -18.5e-3 11e-3" rpy="0 0 0" />
         <geometry>
-          <sphere radius=".03"/>
+          <box size="22e-3 15e-3 20e-3" />
+        </geometry>
+      </collision>
+      <!-- cartriage sledge -->
+      <collision>
+        <origin xyz="0 -6.8e-3 2.2e-3" rpy="0 0 0" />
+        <geometry>
+          <box size="22e-3 8.8e-3 3.8e-3" />
+        </geometry>
+      </collision>
+      <!-- diagonal finger -->
+      <collision>
+        <origin xyz="0 -15.9e-3 28.35e-3" rpy="${-pi/6} 0 0" />
+        <geometry>
+          <box size="17.5e-3 7e-3 23.5e-3" />
+        </geometry>
+      </collision>
+      <!-- rubber tip with which to grasp -->
+      <collision>
+        <origin xyz="0 -7.58e-3 45.25e-3" rpy="0 0 0" />
+        <geometry>
+          <box size="17.5e-3 15.2e-3 18.5e-3" />
         </geometry>
       </collision>

Commit message: Tap tap video

File: urdf/franka_hand.xacro (robot description, xacro)
@@ -35,5 +35,5 @@
       <!-- screw mount -->
       <collision>
-        <origin xyz="0 18.5e-3 11e-3" rpy="0 0 0" />
+        <origin xyz="0 18.5e-3 24e-3" rpy="0 0 0" />
         <geometry>
           <xacro:if value="${pinocchio_collisions}">
@@ -62,5 +62,5 @@
         <!-- rubber tip with which to grasp -->
         <collision>
-          <origin xyz="0 7.58e-3 45.25e-3" rpy="0 0 0" />
+          <origin xyz="0 7.58e-3 45.24e-3" rpy="0 0 0" />
           <geometry>
             <box size="17.5e-3 15.2e-3 18.5e-3" />
@@ -79,5 +79,5 @@
       <!-- screw mount -->
       <collision>
-        <origin xyz="0 -18.5e-3 11e-3" rpy="0 0 0" />
+        <origin xyz="0 -18.5e-3 24e-3" rpy="0 0 0" />
         <geometry>
           <xacro:if value="${pinocchio_collisions}">
@@ -106,5 +106,5 @@
       <!-- rubber tip with which to grasp -->
       <collision>
-        <origin xyz="0 -7.58e-3 45.25e-3" rpy="0 0 0" />
+        <origin xyz="0 -7.58e-3 45.24e-3" rpy="0 0 0" />
         <geometry>
           <box size="17.5e-3 15.2e-3 18.5e-3" />
