Commit message: post treatment

File: post-treatment/models/franka_description/robots/panda/franka2.urdf (robot description, URDF)
Before this commit: robot pandas, 41 links, 40 joints
Links:
- link panda2_leftfinger: geometry collision sphere radius=.03
- link panda2_rightfinger: geometry collision sphere radius=.03
